File: Carte_LCD_FarmingMars/Carte_LCD_FarmingMars.kicad_pcb (KiCad board)
At the start: 2 copper layers, 85 x 60 mm, 22 parts, among them J2 Conn_01x02_Pin, J3 Conn_01x04_Pin, J4 Conn_01x02_Pin, SW1 SW_Push, SW2 SW_Push, SW3 SW_Push, U1 3V3 reg, U2 ATtiny1616-S

Commit message: release V1
Parts:
- added H1: MountingHole, MountingHole:MountingHole_3.2mm_M3, F.Cu at (89.0, 77.0)
- added H2: MountingHole, MountingHole:MountingHole_3.2mm_M3, F.Cu at (105.5, 127.0)
- added H3: MountingHole, MountingHole:MountingHole_3.2mm_M3, F.Cu at (153.0, 77.0)
- added H4: MountingHole, MountingHole:MountingHole_3.2mm_M3, F.Cu at (149.5, 127.0)
- moved SW3 2.28 mm to (113.0, 126.9)
- moved D2 1.79 mm to (158.0, 128.5)
- moved R3 1.79 mm to (160.1, 120.9)
- moved R1 1.79 mm to (156.1, 120.9)
- moved R2 1.79 mm to (158.0, 120.9)
Routing:
- net B_OUT: track 32.2 -> 30.1 mm
- net GREEN: track 60.4 -> 62.2 mm
- net RED: track 74.5 -> 76.3 mm
- net BLUE: track 53.6 -> 54.9 mm
Other:
- board size 85 x 60 mm -> 85 x 62 mm
