File: Carte_LCD_FarmingMars/Carte_LCD_FarmingMars.kicad_sch (KiCad schematic)
At the start: 17 parts, among them J2 Conn_01x02_Pin, J3 Conn_01x04_Pin, SW1 SW_DIP_x01, SW2 SW_Push, SW3 SW_Push, U1 3V3 reg, U2 ATtiny1616-S

Commit message: Followed discord changes
Parts:
- added J1: Screw_Terminal_01x02, symbol Connector:Screw_Terminal_01x02
- added J4: Conn_01x02_Pin, Connector_PinHeader_2.54mm:PinHeader_1x02_P2.54mm_Horizontal, symbol Connector:Conn_01x02_Pin
- added R2, R3, R4: 470, Resistor_SMD:R_0603_1608Metric, symbol Device:R
- J2: footprint Connector_PinHeader_2.54mm:PinHeader_1x02_P2.54mm_Vertical -> Connector_PinHeader_2.54mm:PinHeader_1x02_P2.54mm_Horizontal
- J3: footprint Connector_PinHeader_2.54mm:PinHeader_1x04_P2.54mm_Vertical -> Connector_PinHeader_2.54mm:PinHeader_1x04_P2.54mm_Horizontal
- R1: value 58 -> 470
Connections:
- net +3.3V: now also RV2.3
- net +5V: now also RV1.3; no longer RV1.1, RV2.1
- net BLUE: now also R3.1; no longer D2.4 (BA)
- net GND: now also RV1.1, RV2.1, J1.1 (Pin_1), J4.2 (Pin_2); no longer RV1.3, RV2.3
- net GREEN: now also R2.1; no longer D2.5 (GA)
- net at U2.16 (~{RESET}/PA0): now also R4.1
- net +BATT renamed ALIM 5V
- net ALIM 5V: now also J1.2 (Pin_2)
- new net: D2.4 (BA), R3.2
- new net: D2.5 (GA), R2.2
- new net UPDI: J4.1 (Pin_1), R4.2
- no-connect marks 5 -> 4
Other:
- moved on the sheet: BZ1, R_Buzz1

Commit message: Placement préliminaire PCB
Parts:
- J1: footprint (none) -> ENAC_robotique:Bornier_2x3.81mm
Changed lines of the file:
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@@
       (effects (font (size 1.27 1.27)))
     )
-    (property "Footprint" "" (at 78.74 34.29 0)
+    (property "Footprint" "ENAC_robotique:Bornier_2x3.81mm" (at 78.74 34.29 0)
       (effects (font (size 1.27 1.27)) hide)
     )

Commit message: placement composants
Parts:
- removed J1: Screw_Terminal_01x02, ENAC_robotique:Bornier_2x3.81mm, symbol Connector:Screw_Terminal_01x02
Connections:
- net ALIM 5V is gone; now on net +5V: C1.1, U1.1 (IN)
- net D4: now also U2.12 (PC0); no longer U2.15 (PC3)
- net D5: now also U2.13 (PC1); no longer U2.14 (PC2)
- net D6: now also U2.14 (PC2); no longer U2.13 (PC1)
- net D7: now also U2.15 (PC3); no longer U2.12 (PC0)

Commit message: Routage, inversion pin Couleur et Vbuzz
Connections:
- net COULEUR: now also U2.5 (PA7); no longer U2.4 (PA6)
- net VBUZZ: now also U2.4 (PA6); no longer U2.5 (PA7)
Changed lines of the file:
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@@
     )
   )
-  (global_label "COULEUR" (shape input) (at 58.42 110.49 0) (fields_autoplaced)
+  (global_label "COULEUR" (shape input) (at 58.42 113.03 0) (fields_autoplaced)
     (effects (font (size 1.27 1.27)) (justify left))
-    (property "Intersheetrefs" "${INTERSHEET_REFS}" (at 70.1138 110.49 0)
+    (property "Intersheetrefs" "${INTERSHEET_REFS}" (at 70.1138 113.03 0)
       (effects (font (size 1.27 1.27)) (justify left) hide)
     )
@@
     )
   )
-  (global_label "VBUZZ" (shape input) (at 58.42 113.03 0) (fields_autoplaced)
+  (global_label "VBUZZ" (shape input) (at 58.42 110.49 0) (fields_autoplaced)
     (effects (font (size 1.27 1.27)) (justify left))
-    (property "Intersheetrefs" "${INTERSHEET_REFS}" (at 67.5133 113.03 0)
+    (property "Intersheetrefs" "${INTERSHEET_REFS}" (at 67.5133 110.49 0)
       (effects (font (size 1.27 1.27)) (justify left) hide)
     )

Commit message: annotations
Parts:
- removed SW1: SW_DIP_x01, ENAC_robotique:SWITCH_DTSM31NV, symbol Switch:SW_DIP_x01
- added SW1: SW_Push, ENAC_robotique:SWITCH_DTSM31NV, symbol Switch:SW_Push
Connections:
- net B_IN: now also U2.5 (PA7), SW1.1; no longer SW2.1, U2.7 (PB4)
- net COULEUR: now also SW2.1, U2.7 (PB4); no longer U2.5 (PA7)
- net GND: now also SW1.2
Other:
- moved on the sheet: SW2

Commit message: release V1
Parts:
- added H1, H2, H3, H4: MountingHole, MountingHole:MountingHole_3.2mm_M3, symbol Mechanical:MountingHole
